Commit message: 正常训练，只是步态有问题，不能实物部署

File: resources/robots/bot_elf/urdf/bot_elf_fixarm.urdf (robot description, URDF)
Before this commit: robot bot_elf, 24 links, 23 joints
Links:
- link l_elb_y_link: geometry visual mesh filename=../meshes/l_elb_y_link.STL
- link r_elb_y_link: geometry visual mesh filename=../meshes/r_elb_y_link.STL
Joints:
- joint l_elb_y_joint: type revolute -> fixed
- joint l_shld_x_joint: type revolute -> fixed
- joint l_shld_y_joint: type revolute -> fixed
- joint l_shld_z_joint: type revolute -> fixed
- joint r_elb_y_joint: type revolute -> fixed
- joint r_shld_x_joint: type revolute -> fixed
- joint r_shld_y_joint: type revolute -> fixed
- joint r_shld_z_joint: type revolute -> fixed

Commit message: 训练，正常步态的模型

File: resources/robots/bot_elf/urdf/bot_elf_fixarm.urdf (robot description, URDF)
Before this commit: robot bot_elf, 24 links, 23 joints
Links:
- link l_ankle_x_link: geometry collision mesh filename=../meshes/l_ankle_x_link.STL; visual mesh filename=../meshes/l_ankle_x_link.STL
- link l_elb_y_link: geometry collision mesh filename=../meshes/l_elb_y_link.STL; visual mesh filename=../meshes/l_elb_y_link.STL
- link l_shld_y_link: geometry visual mesh filename=../meshes/l_shld_y_link.STL
- link l_shld_z_link: geometry visual mesh filename=../meshes/l_shld_z_link.STL
- link r_ankle_x_link: geometry collision mesh filename=../meshes/r_ankle_x_link.STL; visual mesh filename=../meshes/r_ankle_x_link.STL
- link r_elb_y_link: geometry collision mesh filename=../meshes/r_elb_y_link.STL; visual mesh filename=../meshes/r_elb_y_link.STL
- link r_shld_y_link: geometry visual mesh filename=../meshes/r_shld_y_link.STL
- link r_shld_z_link: geometry visual mesh filename=../meshes/r_shld_z_link.STL
Joints:
- joint l_elb_y_joint: origin xyz=0 0 -0.24505 rpy=0 0 0 -> xyz=0 0 -0.24505 rpy=0 -1.2 0
- joint l_shld_x_joint: origin xyz=0 0 0 rpy=0 0 0 -> xyz=0 0 0 rpy=0.1 0 0
- joint l_shld_y_joint: origin xyz=0 0.213 0.1521 rpy=0 0 0 -> xyz=0 0.213 0.1521 rpy=0 0.5 0
- joint r_elb_y_joint: origin xyz=0 0 -0.24505 rpy=0 0 0 -> xyz=0 0 -0.24505 rpy=0 -1.2 0
- joint r_shld_x_joint: origin xyz=0 0 0 rpy=0 0 0 -> xyz=0 0 0 rpy=-0.1 0 0
- joint r_shld_y_joint: origin xyz=0 -0.213 0.1521 rpy=0 0 0 -> xyz=0 -0.213 0.1521 rpy=0 0.5 0
