Commit message: 更换bot_elf模型

File: resources/robots/bot_elf/urdf/bot_elf.urdf (robot description, URDF)
Before this commit: robot bot_elf, 32 links, 31 joints
Links:
- removed link contact1
- removed link contact2
- removed link contact3
- removed link contact4
- removed link contact5
- removed link contact6
- removed link contact7
- removed link contact8
- link base_link: mass 8.1797 -> 8.50938212; geometry collision mesh filename=../meshes/base_link.STL; visual mesh filename=../meshes/base_link.STL
- link l_ankle_x_link: mass 0.242076229237956 -> 0.36482443; geometry collision cylinder length=0.16 radius=0.02; collision cylinder length=0.16 radius=0.02
- link l_ankle_y_link: mass 0.0230716180694964 -> 0.02307162; geometry visual mesh filename=../meshes/l_ankle_y_link.STL
- link l_elb_y_link: mass 0.164832849485564 -> 0.16483285; geometry collision mesh filename=../meshes/l_elb_y_link.STL; visual mesh filename=../meshes/l_elb_y_link.STL
- link l_hip_x_link: mass 1.52690683733997 -> 1.74956721; geometry visual mesh filename=../meshes/l_hip_x_link.STL
- link l_hip_y_link: mass 2.50086507860377 -> 2.500865; geometry collision mesh filename=../meshes/l_hip_y_link.STL; visual mesh filename=../meshes/l_hip_y_link.STL
- link l_hip_z_link: mass 1.23681233828303 -> 1.23681234; geometry visual mesh filename=../meshes/l_hip_z_link.STL
- link l_knee_y_link: mass 1.42611317447382 -> 1.58922365; geometry collision cylinder length=0.15 radius=0.035; visual mesh filename=../meshes/l_knee_y_link.STL
- link l_shld_x_link: mass 0.621968051279973 -> 0.62196805; geometry collision mesh filename=../meshes/l_shld_x_link.STL; visual mesh filename=../meshes/l_shld_x_link.STL
- link l_shld_y_link: mass 0.397430898254414 -> 0.3974309; geometry collision mesh filename=../meshes/l_shld_y_link.STL; visual mesh filename=../meshes/l_shld_y_link.STL
- link l_shld_z_link: mass 0.449112448185888 -> 0.44911245; geometry collision mesh filename=../meshes/l_shld_z_link.STL; visual mesh filename=../meshes/l_shld_z_link.STL
- link r_ankle_x_link: mass 0.24207626222516 -> 0.36482447; geometry collision cylinder length=0.16 radius=0.02; collision cylinder length=0.16 radius=0.02
- link r_ankle_y_link: mass 0.0230716180694967 -> 0.02307162; geometry visual mesh filename=../meshes/r_ankle_y_link.STL
- link r_elb_y_link: mass 0.164832849485564 -> 0.16483285; geometry collision mesh filename=../meshes/r_elb_y_link.STL; visual mesh filename=../meshes/r_elb_y_link.STL
- link r_hip_x_link: mass 1.52690683726889 -> 1.74956721; geometry visual mesh filename=../meshes/r_hip_x_link.STL
- link r_hip_y_link: mass 2.50086518492187 -> 2.50086544; geometry collision mesh filename=../meshes/r_hip_y_link.STL; visual mesh filename=../meshes/r_hip_y_link.STL
- link r_hip_z_link: mass 1.23681232467206 -> 1.23681233; geometry visual mesh filename=../meshes/r_hip_z_link.STL
- link r_knee_y_link: mass 1.42506790131187 -> 1.5881784; geometry collision cylinder length=0.15 radius=0.035; visual mesh filename=../meshes/r_knee_y_link.STL
- link r_shld_x_link: mass 0.621968051279973 -> 0.62196805; geometry collision mesh filename=../meshes/r_shld_x_link.STL; visual mesh filename=../meshes/r_shld_x_link.STL
- link r_shld_y_link: mass 0.397430898254414 -> 0.39742959; geometry collision mesh filename=../meshes/r_shld_y_link.STL; visual mesh filename=../meshes/r_shld_y_link.STL
- link r_shld_z_link: mass 0.449113232804568 -> 0.44911323; geometry collision mesh filename=../meshes/r_shld_z_link.STL; visual mesh filename=../meshes/r_shld_z_link.STL
Joints:
- removed joint contact1_joint
- removed joint contact2_joint
- removed joint contact3_joint
- removed joint contact4_joint
- removed joint contact5_joint
- removed joint contact6_joint
- removed joint contact7_joint
- removed joint contact8_joint
- joint l_ankle_x_joint: limit lower=-0.349 upper=0.349 effort=14 velocity=20 -> lower=-0.349 upper=0.349 effort=5 velocity=20
- joint l_ankle_y_joint: limit lower=-1.134 upper=0.872 effort=14 velocity=20 -> lower=-1.134 upper=0.872 effort=10 velocity=20
- joint l_elb_y_joint: limit lower=-2 upper=2 effort=27 velocity=20 -> lower=-2 upper=0 effort=27 velocity=20
- joint l_hip_x_joint: limit lower=-0.523 upper=0.785 effort=40 velocity=20 -> lower=-0.523 upper=0.785 effort=38 velocity=20
- joint l_hip_y_joint: limit lower=-2 upper=0.5 effort=150 velocity=20 -> lower=-2 upper=0.5 effort=80 velocity=20
- joint l_hip_z_joint: limit lower=-0.785 upper=0.785 effort=20 velocity=20 -> lower=-0.785 upper=0.785 effort=18 velocity=20
- joint l_knee_y_joint: limit lower=0 upper=2.2 effort=150 velocity=20 -> lower=0 upper=2.2 effort=100 velocity=20
- joint l_shld_x_joint: limit lower=-0.2 upper=3.14 effort=27 velocity=20 -> lower=-0.52 upper=2 effort=27 velocity=20
- joint l_shld_y_joint: limit lower=-2 upper=2 effort=27 velocity=20 -> lower=-1.5 upper=1.5 effort=27 velocity=20
- joint l_shld_z_joint: limit lower=-2 upper=2 effort=7 velocity=20 -> lower=-1.5 upper=1.5 effort=7 velocity=20
- joint r_ankle_x_joint: limit lower=-0.349 upper=0.349 effort=14 velocity=20 -> lower=-0.349 upper=0.349 effort=5 velocity=20
- joint r_ankle_y_joint: limit lower=-1.134 upper=0.872 effort=14 velocity=20 -> lower=-1.134 upper=0.872 effort=10 velocity=20
- joint r_elb_y_joint: limit lower=-2 upper=2 effort=27 velocity=20 -> lower=-2 upper=0 effort=27 velocity=20
- joint r_hip_x_joint: limit lower=-0.785 upper=0.523 effort=40 velocity=20 -> lower=-0.785 upper=0.523 effort=38 velocity=20
- joint r_hip_y_joint: limit lower=-2 upper=0.5 effort=150 velocity=20 -> lower=-2 upper=0.5 effort=80 velocity=20
- joint r_hip_z_joint: limit lower=-0.785 upper=0.785 effort=20 velocity=20 -> lower=-0.785 upper=0.785 effort=18 velocity=20
- joint r_knee_y_joint: limit lower=0 upper=2.2 effort=150 velocity=20 -> lower=0 upper=2.2 effort=100 velocity=20
- joint r_shld_x_joint: limit lower=-3.14 upper=0.2 effort=27 velocity=20 -> lower=-2 upper=0.52 effort=27 velocity=20
- joint r_shld_y_joint: limit lower=-2 upper=2 effort=27 velocity=20 -> lower=-1.5 upper=1.5 effort=27 velocity=20
- joint r_shld_z_joint: limit lower=-2 upper=2 effort=7 velocity=20 -> lower=-1.5 upper=1.5 effort=7 velocity=20

Commit message: 带有手臂的训练

File: resources/robots/bot_elf/urdf/bot_elf.urdf (robot description, URDF)
Before this commit: robot bot_elf, 24 links, 23 joints
Links:
- link l_ankle_x_link: geometry collision mesh filename=../meshes/l_ankle_x_link.STL; visual mesh filename=../meshes/l_ankle_x_link.STL
- link l_shld_y_link: geometry visual mesh filename=../meshes/l_shld_y_link.STL
- link l_shld_z_link: geometry visual mesh filename=../meshes/l_shld_z_link.STL
- link r_ankle_x_link: geometry collision mesh filename=../meshes/r_ankle_x_link.STL; visual mesh filename=../meshes/r_ankle_x_link.STL
- link r_shld_y_link: geometry visual mesh filename=../meshes/r_shld_y_link.STL
- link r_shld_z_link: geometry visual mesh filename=../meshes/r_shld_z_link.STL
